Commit message: Modified the wheel inertias

File: robot_description/urdf/robot.xacro (robot description, xacro)
@@ -7,5 +7,5 @@
 	<xacro:property name="robot_caster_wheel_radius" value="0.05"/>
 	<xacro:property name="robot_caster_wheel_radius_collision" value="0.0499"/>
-	<xacro:property name="robot_wheel_mass" value="5"/>
+	<xacro:property name="robot_wheel_mass" value="1"/>
 	<xacro:property name="robot_wheel_length" value="0.02"/>
 	<xacro:property name="robot_wheel_radius" value="0.075"/>
@@ -20,5 +20,5 @@
 			<mass value="${robot_chassis_mass}"/>
       		<origin xyz="0.0 0 0" rpy=" 0 0 0"/>
-      		<inertia ixx="0.147116667" ixy="0" ixz="0" iyy="0.334951167" iyz="0" izz="0.3978345"/></inertial>
+      		<inertia ixx="0.147116667" ixy="0" ixz="0" iyy="0.304951167" iyz="0" izz="0.3978345"/></inertial>
 		<collision name="collision">
 			<origin xyz="0 0 0.0" rpy=" 0 0 0"/>
@@ -40,7 +40,7 @@
 			<origin xyz="0 0 0" rpy="0 1.5707 1.5707"/>
 			<inertia
-				ixx="0.1" ixy="0.0" ixz="0.0"
-				iyy="0.1" iyz="0.0"
-				izz="0.1"
+				ixx="0.05" ixy="0.0" ixz="0.0"
+				iyy="0.01" iyz="0.0"
+				izz="0.01"
 			/>
 		</inertial>
@@ -64,7 +64,7 @@
 			<origin xyz="0 0 0" rpy="0 1.5707 1.5707"/>
 			<inertia
-				ixx="0.1" ixy="0.0" ixz="0.0"
-				iyy="0.1" iyz="0.0"
-				izz="0.1"
+				ixx="0.05" ixy="0.0" ixz="0.0"
+				iyy="0.01" iyz="0.0"
+				izz="0.01"
 			/>
 		</inertial>
@@ -88,7 +88,7 @@
 			<origin xyz="0 0 0" rpy="0 1.5707 1.5707"/>
 			<inertia
-				ixx="0.1" ixy="0.0" ixz="0.0"
-				iyy="0.1" iyz="0.0"
-				izz="0.1"
+				ixx="0.05" ixy="0.0" ixz="0.0"
+				iyy="0.01" iyz="0.0"
+				izz="0.01"
 			/>
 		</inertial>
@@ -112,7 +112,7 @@
 			<origin xyz="0 0 0" rpy="0 1.5707 1.5707"/>
 			<inertia
-				ixx="0.1" ixy="0.0" ixz="0.0"
-				iyy="0.1" iyz="0.0"
-				izz="0.1"
+				ixx="0.05" ixy="0.0" ixz="0.0"
+				iyy="0.01" iyz="0.0"
+				izz="0.01"
 			/>
 		</inertial>
